File: M.2.kicad_sch (KiCad schematic)
At the start: 3 parts, among them J1 Bus_M.2_Socket_B

Commit message: second version
Connections:
- net USB_2_P4+ renamed USB_2_P1+
Changed lines of the file:
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@@
 		)
 	)
-	(hierarchical_label "USB_2_P4+"
+	(hierarchical_label "USB_2_P1+"
 		(shape bidirectional)
 		(at 54.61 77.47 180)
